File: hardware/imu_to_dxl/imu_to_dxl.kicad_pcb (KiCad board)
At the start: 2 copper layers, 27.1 x 30.2 mm, 74 parts, among them CN1 B3B-EH-A (LF)(SN), CN2 B3B-PH-K-S(LF)(SN), J1 1.8mm螺丝孔, J2 1.8mm螺丝孔, J3 1.8mm螺丝孔, J4 1.8mm螺丝孔, Q1 MMBT3906, U1 ETA2845S2G_C22362741, U2 GD32F303CCT6, U3 LSM6DSV16XTR, U4 SN74LVC1G126DBVR, U5 SN74LVC1G125DBV, U6 ME6211C18M5G-N, X1 XL2EL89CSI-111YLC-12M

Commit message: update: BOM
Parts:
- CN1: value B3B-EH-A (LF)(SN) -> ~
- CN2: value B3B-PH-K-S(LF)(SN) -> ~
Changed lines of the file:
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@@
 			)
 		)
-		(property "Value" "B3B-PH-K-S(LF)(SN)"
+		(property "Value" "~"
 			(at 0.03 2.662 0)
 			(layer "F.Fab")
@@
 		(sheetname "/")
 		(sheetfile "imu_to_dxl.kicad_sch")
+		(attr exclude_from_bom dnp)
 		(fp_line
 			(start -4 -1.6)
@@
 			)
 		)
-		(property "Value" "B3B-EH-A (LF)(SN)"
+		(property "Value" "~"
 			(at 0.0251 3.162 0)
 			(layer "F.Fab")
@@
 		(sheetname "/")
 		(sheetfile "imu_to_dxl.kicad_sch")
+		(attr exclude_from_bom dnp)
 		(fp_line
 			(start -4.9999 -1.6001)
@@
 			)
 		)
-		(property "Manufacturer Part" "JK-SMD0603-002"
+		(property "Manufacturer Part" "JK-SMD0603-001"
 			(at 0 0 270)
 			(unlocked yes)
@@
 			)
 		)
-		(property "LCSC Part" "C1884486"
+		(property "LCSC Part" "C2687114"
 			(at 0 0 270)
 			(unlocked yes)

Commit message: 更新原理和PCB，优化飞特舵机上拉电阻小导致小概率丢包问题
Parts:
- D2: value 3.3V ESD -> 5V ESD
- R31: value 10k -> 100k
- R5: value 100R -> 51R
