File: hardware/imu_to_dxl/imu_to_dxl.kicad_pcb (KiCad board)
At the start: 2 copper layers, 27.1 x 30.2 mm, 77 parts, among them CN1 B3B-EH-A(LF)(SN), CN2 AMP175778/8283/A2007WV-3P, J1 1.8mm螺丝孔, J2 1.8mm螺丝孔, J3 1.8mm螺丝孔, J4 1.8mm螺丝孔, Q1 MMBT3906, U1 ETA2845S2G_C22362741, U2 GD32F303CCT6, U3 LSM6DSV16XTR, U4 SN74LVC1G126DBVR, U5 SN74LVC1G125DBV, U6 ME6211C18M5G-N, X1 XL2EL89CSI-111YLC-12M

Commit message: update bom
Parts:
- C17: value 27pF/50V -> 20pF/50V
- R34: value 100K -> 1K
- turned R34 to -90 degrees
Connections:
- R34 pad 1: Net-(LED1-K) -> GND
- R34 pad 2: GND -> Net-(LED1-K)
