File: hardware/imu_to_dxl/imu_to_dxl.kicad_sch (KiCad schematic)
At the start: 74 parts, among them CN1 B3B-EH-A (LF)(SN), CN2 B3B-PH-K-S(LF)(SN), J1 1.8mm螺丝孔, J2 1.8mm螺丝孔, J3 1.8mm螺丝孔, J4 1.8mm螺丝孔, Q1 MMBT3906, U1 ETA2845S2G_C22362741, U2 GD32F303CCT6, U3 LSM6DSV16XTR, U4 SN74LVC1G126DBVR, U5 SN74LVC1G125DBV, U6 ME6211C18M5G-N, X1 XL2EL89CSI-111YLC-12M

Commit message: update: readme
Parts:
- F1: LCSC Part C1884486 -> C2687114; Manufacturer Part JK-SMD0603-002 -> JK-SMD0603-001
Other:
- note removed: "改为JK-SMD0603-001"
Changed lines of the file:
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@@
-		)
-	)
-	(text "改为JK-SMD0603-001"
-		(exclude_from_sim no)
-		(at 89.662 31.75 0)
-		(effects
-			(font
-				(size 1.27 1.27)
-			)
 		)
 	)
@@
 			)
 		)
-		(property "Manufacturer Part" "JK-SMD0603-002"
+		(property "Manufacturer Part" "JK-SMD0603-001"
 			(at 87.63 29.21 0)
 			(effects
@@
 			)
 		)
-		(property "LCSC Part" "C1884486"
+		(property "LCSC Part" "C2687114"
 			(at 87.63 29.21 0)
 			(effects

Commit message: update: BOM
Parts:
- CN1: value B3B-EH-A (LF)(SN) -> ~; LCSC Part C160259 -> (none); Manufacturer JST -> (none); Manufacturer Part B3B-EH-A(LF)(SN) -> (none); Supplier LCSC -> (none); now not fitted; now left out of the parts list
- CN2: value B3B-PH-K-S(LF)(SN) -> ~; LCSC Part C131339 -> (none); Manufacturer JST -> (none); Manufacturer Part B3B-PH-K-S(LF)(SN) -> (none); Supplier LCSC -> (none); now not fitted; now left out of the parts list
Other:
- note added: "二选一，手工焊接"
Changed lines of the file:
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@@
 		)
 	)
+	(text "二选一，手工焊接"
+		(exclude_from_sim no)
+		(at 45.466 34.544 0)
+		(effects
+			(font
+				(size 1.27 1.27)
+			)
+		)
+	)
 	(text "SWD"
 		(exclude_from_sim no)
@@
 		(unit 1)
 		(exclude_from_sim no)
-		(in_bom yes)
+		(in_bom no)
 		(on_board yes)
-		(dnp no)
+		(dnp yes)
 		(property "Reference" "CN2"
 			(at 40.64 43.1801 0)
@@
 			)
 		)
-		(property "Value" "B3B-PH-K-S(LF)(SN)"
+		(property "Value" "~"
 			(at 40.64 40.6401 0)
 			(effects
@@
 			)
 		)
-		(property "Manufacturer Part" "B3B-PH-K-S(LF)(SN)"
-			(at 44.45 41.91 0)
-			(effects
-				(font
-					(size 1.27 1.27)
-				)
-				(hide yes)
-			)
-		)
-		(property "Manufacturer" "JST"
-			(at 44.45 41.91 0)
-			(effects
-				(font
-					(size 1.27 1.27)
-				)
-				(hide yes)
-			)
-		)
-		(property "LCSC Part" "C131339"
-			(at 44.45 41.91 0)
-			(effects
-				(font
-					(size 1.27 1.27)
-				)
-				(hide yes)
-			)
-		)
-		(property "Supplier" "LCSC"
-			(at 44.45 41.91 0)
-			(effects
-				(font
-					(size 1.27 1.27)
-				)
-				(hide yes)
-			)
-		)
 		(pin "1"
 		)
@@
 		(unit 1)
 		(exclude_from_sim no)
-		(in_bom yes)
+		(in_bom no)
 		(on_board yes)
-		(dnp no)
+		(dnp yes)
 		(fields_autoplaced yes)
 		(property "Reference" "CN1"
@@
 			)
 		)
-		(property "Value" "B3B-EH-A (LF)(SN)"
+		(property "Value" "~"
 			(at 39.37 27.9399 0)
 			(effects
@@
 			(at 46.99 26.67 0)
 			(effects
-				(font
-					(size 1.27 1.27)
-				)
-				(hide yes)
-			)
-		)
-		(property "Manufacturer Part" "B3B-EH-A(LF)(SN)"
-			(at 46.99 26.67 0)
-			(effects
-				(font
-					(size 1.27 1.27)
-				)
-				(hide yes)
-			)
-		)
-		(property "Manufacturer" "JST"
-			(at 46.99 26.67 0)
-			(effects
-				(font
-					(size 1.27 1.27)
-				)
-				(hide yes)
-			)
-		)
-		(property "LCSC Part" "C160259"
-			(at 46.99 26.67 0)
-			(effects
-				(font
-					(size 1.27 1.27)
-				)
-				(hide yes)
-			)
-		)
-		(property "Supplier" "LCSC"
-			(at 46.99 26.67 0)
-			(effects

Commit message: 更新原理和PCB，优化飞特舵机上拉电阻小导致小概率丢包问题
Parts:
- D2: value 3.3V ESD -> 5V ESD; LCSC Part C46551335 -> C19224; Manufacturer SPSEMI(瞬雷电子) -> (none); Manufacturer Part TUSD03FB -> (none)
- R31: value 10k -> 100k; LCSC Part C25744 -> C25741
- R5: value 100R -> 51R; LCSC Part C110091 -> C2907181
Changed lines of the file:
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@@
 			)
 		)
-		(property "Value" "10k"
+		(property "Value" "100k"
 			(at 149.86 106.68 0)
 			(effects
@@
 			)
 		)
-		(property "LCSC Part" "C25744"
+		(property "LCSC Part" "C25741"
 			(at 154.94 107.95 0)
 			(effects
@@
 			)
 		)
-		(property "Value" "100R"
+		(property "Value" "51R"
 			(at 105.41 25.4 0)
 			(effects
@@
 			)
 		)
-		(property "LCSC Part" "C110091"
+		(property "LCSC Part" "C2907181"
 			(at 105.41 29.21 0)
 			(effects
@@
 			)
 		)
-		(property "Value" "3.3V ESD"
+		(property "Value" "5V ESD"
 			(at 102.87 41.9099 90)
 			(effects
@@
 			)
 		)
-		(property "Manufacturer Part" "TUSD03FB"
+		(property "Manufacturer Part" ""
 			(at 96.52 39.37 0)
 			(effects
@@
 			)
 		)
-		(property "Manufacturer" "SPSEMI(瞬雷电子)"
+		(property "Manufacturer" ""
 			(at 96.52 39.37 0)
 			(effects
@@
 			)
 		)
-		(property "LCSC Part" "C46551335"
+		(property "LCSC Part" "C19224"
 			(at 96.52 39.37 0)
 			(effects
