File: hardware/imu_to_dxl/imu_to_dxl.kicad_sch (KiCad schematic)
At the start: 77 parts, among them CN1 B3B-EH-A(LF)(SN), CN2 AMP175778/8283/A2007WV-3P, J1 1.8mm螺丝孔, J2 1.8mm螺丝孔, J3 1.8mm螺丝孔, J4 1.8mm螺丝孔, Q1 MMBT3906, U1 ETA2845S2G_C22362741, U2 GD32F303CCT6, U3 LSM6DSV16XTR, U4 SN74LVC1G126DBVR, U5 SN74LVC1G125DBV, U6 ME6211C18M5G-N, X1 XL2EL89CSI-111YLC-12M

Commit message: update bom
Parts:
- C17: value 27pF/50V -> 20pF/50V; LCSC Part C107002 -> C107000
- LED1: LCSC Part (none) -> C51933293; Supplier Part C51933293 -> (none)
- R34: value 100K -> 1K; LCSC Part C25741 -> C11702
Connections:
- net GND: now also R34.1; no longer R34.2
- net at LED1.1 (K): now also R34.2; no longer R34.1
Changed lines of the file:
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@@
 	)
 	(symbol
+		(lib_name "RC0402FR-0710KL_1")
+		(lib_id "microduck:RC0402FR-0710KL")
+		(at 171.45 219.71 90)
+		(unit 1)
+		(exclude_from_sim no)
+		(in_bom yes)
+		(on_board yes)
+		(dnp no)
+		(property "Reference" "R34"
+			(at 174.752 218.948 90)
+			(effects
+				(font
+					(size 1.27 1.27)
+				)
+			)
+		)
+		(property "Value" "1K"
+			(at 174.244 221.488 90)
+			(effects
+				(font
+					(size 1.27 1.27)
+				)
+			)
+		)
+		(property "Footprint" "microduck:R0402"
+			(at 171.45 219.71 0)
+			(effects
+				(font
+					(size 1.27 1.27)
+				)
+				(hide yes)
+			)
+		)
+		(property "Datasheet" ""
+			(at 171.45 219.71 0)
+			(effects
+				(font
+					(size 1.27 1.27)
+				)
+				(hide yes)
+			)
+		)
+		(property "Description" ""
+			(at 171.45 219.71 0)
+			(effects
+				(font
+					(size 1.27 1.27)
+				)
+				(hide yes)
+			)
+		)
+		(property "Manufacturer Part" ""
+			(at 171.45 219.71 0)
+			(effects
+				(font
+					(size 1.27 1.27)
+				)
+				(hide yes)
+			)
+		)
+		(property "Manufacturer" ""
+			(at 171.45 219.71 0)
+			(effects
+				(font
+					(size 1.27 1.27)
+				)
+				(hide yes)
+			)
+		)
+		(property "LCSC Part" "C11702"
+			(at 171.45 219.71 0)
+			(effects
+				(font
+					(size 1.27 1.27)
+				)
+				(hide yes)
+			)
+		)
+		(property "Supplier" "LCSC"
+			(at 171.45 219.71 0)
+			(effects
+				(font
+					(size 1.27 1.27)
+				)
+				(hide yes)
+			)
+		)
+		(pin "1"
+		)
+		(pin "2"
+		)
+		(instances
+			(project "imu_to_dxl"
+				(path "/9e76362d-8a32-4a28-948c-242ffcf8f16d"
+					(reference "R34")
+					(unit 1)
+				)
+			)
+		)
+	)
+	(symbol
 		(lib_id "Device:R_Small")
 		(at 154.94 107.95 0)
@@
 			)
 		)
-		(property "Value" "27pF/50V"
+		(property "Value" "20pF/50V"
 			(at 294.64 240.0299 90)
 			(effects
@@
 			)
 		)
-		(property "LCSC Part" "C107002"
+		(property "LCSC Part" "C107000"
 			(at 290.83 238.76 0)
 			(effects
@@
 			)
 		)
-		(property "Supplier Part" "C51933293"
+		(property "LCSC Part" "C51933293"
 			(at 171.45 207.01 0)
 			(effects
@@
 					(unit 1)
 				)
-			)
-		)
-	)
-	(symbol
-		(lib_name "RC0402FR-0710KL_1")
-		(lib_id "microduck:RC0402FR-0710KL")
-		(at 171.45 219.71 270)
-		(unit 1)
-		(exclude_from_sim no)
-		(in_bom yes)
-		(on_board yes)
-		(dnp no)
-		(fields_autoplaced yes)
-		(property "Reference" "R34"
-			(at 173.99 218.4399 90)
-			(effects
-				(font
-					(size 1.27 1.27)
-				)
-				(justify left)
-			)
-		)
-		(property "Value" "100K"
-			(at 173.99 220.9799 90)
-			(effects
-				(font
-					(size 1.27 1.27)
-				)
-				(justify left)
-			)
-		)
-		(property "Footprint" "microduck:R0402"
-			(at 171.45 219.71 0)
-			(effects
-				(font
-					(size 1.27 1.27)
-				)
-				(hide yes)
-			)
-		)
-		(property "Datasheet" ""
-			(at 171.45 219.71 0)
-			(effects
-				(font
-					(size 1.27 1.27)
-				)
-				(hide yes)
-			)
-		)
-		(property "Description" ""
-			(at 171.45 219.71 0)
-			(effects
-				(font
-					(size 1.27 1.27)
-				)
-				(hide yes)
-			)
-		)
-		(property "Manufacturer Part" ""
-			(at 171.45 219.71 0)
-			(effects
-				(font
-					(size 1.27 1.27)
-				)
-				(hide yes)
-			)
-		)
-		(property "Manufacturer" ""
-			(at 171.45 219.71 0)
-			(effects
-				(font
-					(size 1.27 1.27)
-				)
-				(hide yes)
-			)
-		)
-		(property "LCSC Part" "C25741"
-			(at 171.45 219.71 0)
-			(effects
-				(font
-					(size 1.27 1.27)
-				)
-				(hide yes)
-			)
-		)
-		(property "Supplier" "LCSC"
-			(at 171.45 219.71 0)
-			(effects
-				(font
-					(size 1.27 1.27)
-				)
-				(hide yes)
-			)
-		)
-		(pin "1"
-		)
-		(pin "2"
-		)
-		(instances
-			(project "imu_to_dxl"
-				(path "/9e76362d-8a32-4a28-948c-242ffcf8f16d"
-					(reference "R34")
-					(unit 1)
-				)
